File: Ampel/treiber.brd (EAGLE design)
At the start: 35.6 x 35.6 mm, 11 parts, among them IC1 MC34063AP

Commit message: R_SENSE angepasst
Parts:
- R_SENSE: value 0.22R -> 0.18R
Changed lines of the file:
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@@
 <element name="D1" library="diode" package="DO35-7" value="MBRS240" x="16.51" y="13.97" rot="R90"/>
 <element name="R2" library="resistor" package="0207/10" value="47R" x="13.97" y="13.97" rot="R90"/>
-<element name="R_SENSE" library="resistor" package="0207/10" value="0.22R" x="11.43" y="13.97" rot="R90"/>
+<element name="R_SENSE" library="resistor" package="0207/10" value="0.18R" x="11.43" y="13.97" rot="R90"/>
 <element name="L1" library="inductors" package="DR1030" value="220µ" x="26.67" y="12.7" rot="MR180"/>
 <element name="LED" library="pinhead" package="1X02" value="3W" x="20.32" y="3.81"/>
@@
 <contactref element="D1" pad="A"/>
 <contactref element="IC1" pad="1"/>
-<wire x1="16.51" y1="17.78" x2="26.67" y2="17.78" width="0.8128" layer="16"/>
 <wire x1="26.67" y1="17.78" x2="26.67" y2="17.15" width="0.4064" layer="16"/>
 <via x="31.75" y="17.78" extent="1-16" drill="0.8"/>
@@
 <wire x1="21.59" y1="21.59" x2="16.51" y2="21.59" width="0.8128" layer="16"/>
 <wire x1="16.51" y1="21.59" x2="16.51" y2="17.78" width="0.8128" layer="16"/>
+<wire x1="16.51" y1="17.78" x2="26.67" y2="17.78" width="0.8128" layer="16"/>
 </signal>
 <signal name="N$6">

Commit message: Schaltung nochmal angepasst
Parts:
- removed R2: 47R, resistor:0207/10
- C1: device resistor:C075-032X103 -> resistor:C050-024X044
- R_SENSE: device resistor:0207/10 -> resistor:0411/15
- moved C1 3.81 mm to (25.4, 29.2), turned to 90 degrees
- moved C2 1.27 mm to (3.81, 19.1)
- moved R_SENSE 1.27 mm to (11.4, 15.2)
- moved SV1 1.27 mm to (5.08, 29.2)
Connections:
- removed net N$5: D1.A, IC1.1, L1.2
- net N$2: now also D1.A, IC1.1, L1.2; no longer R2.2
- net VCC: no longer R2.1
Routing:
- net N$5: track 24.8 -> 0.00 mm, vias 1 -> 0
- net N$2: track 2.54 -> 27.3 mm, vias 0 -> 1
- net GND: track 39.4 -> 34.3 mm
- net VCC: track 36.8 -> 40.6 mm
- net N$1: track 6.35 -> 3.81 mm
- net PWM: track 7.62 -> 8.89 mm
Changed lines of the file:
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@@
 <elements>
 <element name="IC1" library="mc34063" package="DIL08" value="MC34063AP" x="17.78" y="25.4" rot="R90"/>
-<element name="SV1" library="con-lstb" package="MA03-1" value="Control" x="6.35" y="29.21" rot="R270">
-<attribute name="OC_NEWARK" value="unknown" x="-26.67" y="11.43" size="1.778" layer="27" rot="R270" display="off"/>
-<attribute name="MPN" value="" x="-26.67" y="11.43" size="1.778" layer="27" rot="R270" display="off"/>
-<attribute name="MF" value="" x="-26.67" y="11.43" size="1.778" layer="27" rot="R270" display="off"/>
-<attribute name="OC_FARNELL" value="unknown" x="-26.67" y="11.43" size="1.778" layer="27" rot="R270" display="off"/>
+<element name="SV1" library="con-lstb" package="MA03-1" value="Control" x="5.08" y="29.21" rot="R270">
+<attribute name="OC_NEWARK" value="unknown" x="-27.94" y="11.43" size="1.778" layer="27" rot="R270" display="off"/>
+<attribute name="MPN" value="" x="-27.94" y="11.43" size="1.778" layer="27" rot="R270" display="off"/>
+<attribute name="MF" value="" x="-27.94" y="11.43" size="1.778" layer="27" rot="R270" display="off"/>
+<attribute name="OC_FARNELL" value="unknown" x="-27.94" y="11.43" size="1.778" layer="27" rot="R270" display="off"/>
 </element>
-<element name="C1" library="resistor" package="C075-032X103" value="330p" x="25.4" y="25.4" rot="R270"/>
+<element name="C1" library="resistor" package="C050-024X044" value="330p" x="25.4" y="29.21" rot="R90"/>
 <element name="R1" library="resistor" package="0207/10" value="4.7K" x="8.89" y="24.13" rot="R90"/>
-<element name="C2" library="resistor" package="E2,5-5" value="68µ" x="5.08" y="19.05" rot="R180"/>
+<element name="C2" library="resistor" package="E2,5-5" value="68µ" x="3.81" y="19.05" rot="R180"/>
 <element name="C3" library="capacitor-wima" package="C5B2.5" value="100n" x="11.43" y="29.21" rot="R90"/>
 <element name="D1" library="diode" package="DO35-7" value="MBRS240" x="16.51" y="13.97" rot="R90"/>
-<element name="R2" library="resistor" package="0207/10" value="47R" x="13.97" y="13.97" rot="R90"/>
-<element name="R_SENSE" library="resistor" package="0207/10" value="0.18R" x="11.43" y="13.97" rot="R90"/>
+<element name="R_SENSE" library="resistor" package="0411/15" value="0.18R" x="11.43" y="15.24" rot="R90"/>
 <element name="L1" library="inductors" package="DR1030" value="220µ" x="26.67" y="12.7" rot="MR180"/>
 <element name="LED" library="pinhead" package="1X02" value="3W" x="20.32" y="3.81"/>
@@
 <contactref element="C3" pad="1"/>
 <contactref element="R_SENSE" pad="1"/>
-<contactref element="R2" pad="1"/>
 <contactref element="R1" pad="1"/>
 <contactref element="D1" pad="C"/>
 <contactref element="IC1" pad="6"/>
 <contactref element="SV1" pad="3"/>
-<wire x1="13.97" y1="8.89" x2="11.43" y2="8.89" width="0.8128" layer="16"/>
-<wire x1="11.43" y1="8.89" x2="8.89" y2="8.89" width="0.8128" layer="16"/>
 <wire x1="11.43" y1="26.67" x2="13.97" y2="26.67" width="0.4064" layer="16"/>
 <wire x1="16.51" y1="10.16" x2="16.51" y2="8.89" width="0.8128" layer="16"/>
-<wire x1="16.51" y1="8.89" x2="13.97" y2="8.89" width="0.8128" layer="16"/>
+<wire x1="11.43" y1="26.67" x2="5.08" y2="26.67" width="0.4064" layer="16"/>
+<wire x1="5.08" y1="19.05" x2="5.08" y2="26.67" width="0.8128" layer="16"/>
+<wire x1="5.08" y1="19.05" x2="8.89" y2="19.05" width="0.8128" layer="16"/>
+<wire x1="11.43" y1="8.89" x2="8.89" y2="8.89" width="0.8128" layer="16"/>
 <wire x1="8.89" y1="8.89" x2="8.89" y2="19.05" width="0.8128" layer="16"/>
-<wire x1="11.43" y1="26.67" x2="6.35" y2="26.67" width="0.4064" layer="16"/>
-<wire x1="6.35" y1="19.05" x2="6.35" y2="26.67" width="0.8128" layer="16"/>
-<wire x1="6.35" y1="19.05" x2="8.89" y2="19.05" width="0.8128" layer="16"/>
+<wire x1="11.43" y1="7.62" x2="11.43" y2="8.89" width="0.8128" layer="16"/>
+<wire x1="11.43" y1="8.89" x2="16.51" y2="8.89" width="0.8128" layer="16"/>
 </signal>
 <signal name="PWM">
@@
 <wire x1="13.97" y1="29.21" x2="8.89" y2="29.21" width="0.4064" layer="16"/>
 <contactref element="SV1" pad="2"/>
-<wire x1="6.35" y1="29.21" x2="8.89" y2="29.21" width="0.4064" layer="16"/>
+<wire x1="5.08" y1="29.21" x2="8.89" y2="29.21" width="0.4064" layer="16"/>
 </signal>
 <signal name="GND">
@@
 <wire x1="19.05" y1="29.21" x2="19.05" y2="24.13" width="0.4064" layer="16"/>
 <wire x1="19.05" y1="24.13" x2="21.59" y2="24.13" width="0.4064" layer="16"/>
-<wire x1="6.35" y1="31.75" x2="19.05" y2="31.75" width="0.4064" layer="16"/>
+<wire x1="5.08" y1="31.75" x2="19.05" y2="31.75" width="0.4064" layer="16"/>
 <wire x1="19.05" y1="31.75" x2="19.05" y2="29.21" width="0.4064" layer="16"/>
-<wire x1="11.43" y1="31.75" x2="6.35" y2="31.75" width="0.4064" layer="16"/>
-<wire x1="3.81" y1="31.75" x2="6.35" y2="31.75" width="0.4064" layer="16"/>
-<polygon width="0.4064" layer="16" spacing="0.6096" isolate="0.6096" thermals="no">
+<wire x1="11.43" y1="31.75" x2="5.08" y2="31.75" width="0.4064" layer="16"/>
+<wire x1="3.81" y1="31.75" x2="5.08" y2="31.75" width="0.4064" layer="16"/>
+<polygon width="0.4064" layer="16" spacing="0.6096" isolate="0.6096" orphans="yes">
 <vertex x="0" y="35.56"/>
 <vertex x="0" y="0"/>
@@
 <vertex x="35.56" y="35.56"/>
 </polygon>
-<wire x1="25.4" y1="21.59" x2="25.4" y2="24.13" width="0.4064" layer="16"/>
-<wire x1="25.4" y1="24.13" x2="21.59" y2="24.13" width="0.4064" layer="16"/>
 </signal>
 <signal name="N$1">
 <contactref element="IC1" pad="3"/>
 <contactref element="C1" pad="1"/>
-<wire x1="25.4" y1="29.21" x2="25.4" y2="26.67" width="0.4064" layer="16"/>
-<wire x1="25.4" y1="26.67" x2="21.59" y2="26.67" width="0.4064" layer="16"/>
-</signal>
-<signal name="N$2">
-<contactref element="IC1" pad="8"/>
-<contactref element="R2" pad="2"/>
-<wire x1="13.97" y1="21.59" x2="13.97" y2="19.05" width="0.8128" layer="16"/>
+<wire x1="21.59" y1="26.67" x2="25.4" y2="26.67" width="0.8128" layer="16"/>
 </signal>
 <signal name="N$3">
 <contactref element="R_SENSE" pad="2"/>
-<wire x1="11.43" y1="19.05" x2="11.43" y2="12.7" width="0.8128" layer="16"/>
+<wire x1="11.43" y1="22.86" x2="11.43" y2="12.7" width="0.8128" layer="16"/>
 <wire x1="11.43" y1="12.7" x2="19.05" y2="12.7" width="0.8128" layer="16"/>
-<wire x1="11.43" y1="24.13" x2="11.43" y2="19.05" width="0.8128" layer="16"/>
+<wire x1="11.43" y1="24.13" x2="11.43" y2="22.86" width="0.8128" layer="16"/>
 <contactref element="IC1" pad="7"/>
 <wire x1="11.43" y1="24.13" x2="13.97" y2="24.13" width="0.8128" layer="16"/>
 <contactref element="LED" pad="1"/>
 <wire x1="19.05" y1="3.81" x2="19.05" y2="12.7" width="0.8128" layer="16"/>
-</signal>
-<signal name="N$5">
-<contactref element="L1" pad="2"/>
-<contactref element="D1" pad="A"/>
-<contactref element="IC1" pad="1"/>
-<wire x1="26.67" y1="17.78" x2="26.67" y2="17.15" width="0.4064" layer="16"/>
-<via x="31.75" y="17.78" extent="1-16" drill="0.8"/>
-<wire x1="26.67" y1="17.78" x2="31.75" y2="17.78" width="0.8128" layer="16"/>
-<wire x1="21.59" y1="21.59" x2="16.51" y2="21.59" width="0.8128" layer="16"/>
-<wire x1="16.51" y1="21.59" x2="16.51" y2="17.78" width="0.8128" layer="16"/>
-<wire x1="16.51" y1="17.78" x2="26.67" y2="17.78" width="0.8128" layer="16"/>
 </signal>
 <signal name="N$6">
@@
 <via x="31.75" y="7.62" extent="1-16" drill="0.8"/>
 </signal>
+<signal name="N$2">
+<contactref element="IC1" pad="8"/>
+<contactref element="IC1" pad="1"/>
+<contactref element="L1" pad="2"/>
+<contactref element="D1" pad="A"/>
+<wire x1="26.67" y1="17.78" x2="26.67" y2="17.15" width="0.4064" layer="16"/>
+<via x="31.75" y="17.78" extent="1-16" drill="0.8"/>
+<wire x1="26.67" y1="17.78" x2="31.75" y2="17.78" width="0.8128" layer="16"/>
+<wire x1="16.51" y1="21.59" x2="16.51" y2="17.78" width="0.8128" layer="16"/>
+<wire x1="16.51" y1="17.78" x2="26.67" y2="17.78" width="0.8128" layer="16"/>
+<wire x1="13.97" y1="21.59" x2="21.59" y2="21.59" width="0.8128" layer="16"/>
+<wire x1="13.97" y1="21.59" x2="16.51" y2="21.59" width="0" layer="19" extent="16-16"/>
+</signal>
 </signals>
