File: Ampel/treiber.sch (EAGLE design)
At the start: 11 parts, among them IC1 MC34063AP

Commit message: Pad-Größen und Leiterbahnbreiten angepasst
Other:
- moved on the sheet: D1
Changed lines of the file:
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@@
 <grid distance="0.1" unitdist="inch" unit="inch" style="lines" multiple="1" display="no" altdistance="0.01" altunitdist="inch" altunit="inch"/>
 <layers>
-<layer number="1" name="Top" color="4" fill="1" visible="yes" active="no"/>
-<layer number="16" name="Bottom" color="1" fill="1" visible="yes" active="no"/>
-<layer number="17" name="Pads" color="2" fill="1" visible="yes" active="no"/>
-<layer number="18" name="Vias" color="2" fill="1" visible="yes" active="no"/>
-<layer number="19" name="Unrouted" color="6" fill="1" visible="yes" active="no"/>
-<layer number="20" name="Dimension" color="15" fill="1" visible="yes" active="no"/>
-<layer number="21" name="tPlace" color="7" fill="1" visible="yes" active="no"/>
-<layer number="22" name="bPlace" color="7" fill="1" visible="yes" active="no"/>
-<layer number="23" name="tOrigins" color="15" fill="1" visible="yes" active="no"/>
-<layer number="24" name="bOrigins" color="15" fill="1" visible="yes" active="no"/>
-<layer number="25" name="tNames" color="7" fill="1" visible="yes" active="no"/>
-<layer number="26" name="bNames" color="7" fill="1" visible="yes" active="no"/>
-<layer number="27" name="tValues" color="7" fill="1" visible="yes" active="no"/>
-<layer number="28" name="bValues" color="7" fill="1" visible="yes" active="no"/>
+<layer number="1" name="Top" color="4" fill="1" visible="no" active="no"/>
+<layer number="16" name="Bottom" color="1" fill="1" visible="no" active="no"/>
+<layer number="17" name="Pads" color="2" fill="1" visible="no" active="no"/>
+<layer number="18" name="Vias" color="2" fill="1" visible="no" active="no"/>
+<layer number="19" name="Unrouted" color="6" fill="1" visible="no" active="no"/>
+<layer number="20" name="Dimension" color="15" fill="1" visible="no" active="no"/>
+<layer number="21" name="tPlace" color="7" fill="1" visible="no" active="no"/>
+<layer number="22" name="bPlace" color="7" fill="1" visible="no" active="no"/>
+<layer number="23" name="tOrigins" color="15" fill="1" visible="no" active="no"/>
+<layer number="24" name="bOrigins" color="15" fill="1" visible="no" active="no"/>
+<layer number="25" name="tNames" color="7" fill="1" visible="no" active="no"/>
+<layer number="26" name="bNames" color="7" fill="1" visible="no" active="no"/>
+<layer number="27" name="tValues" color="7" fill="1" visible="no" active="no"/>
+<layer number="28" name="bValues" color="7" fill="1" visible="no" active="no"/>
 <layer number="29" name="tStop" color="7" fill="3" visible="no" active="no"/>
 <layer number="30" name="bStop" color="7" fill="6" visible="no" active="no"/>
@@
 <layer number="35" name="tGlue" color="7" fill="4" visible="no" active="no"/>
 <layer number="36" name="bGlue" color="7" fill="5" visible="no" active="no"/>
-<layer number="37" name="tTest" color="7" fill="1" visible="yes" active="no"/>
-<layer number="38" name="bTest" color="7" fill="1" visible="yes" active="no"/>
+<layer number="37" name="tTest" color="7" fill="1" visible="no" active="no"/>
+<layer number="38" name="bTest" color="7" fill="1" visible="no" active="no"/>
 <layer number="39" name="tKeepout" color="4" fill="11" visible="no" active="no"/>
 <layer number="40" name="bKeepout" color="1" fill="11" visible="no" active="no"/>
@@
 <layer number="44" name="Drills" color="7" fill="1" visible="no" active="no"/>
 <layer number="45" name="Holes" color="7" fill="1" visible="no" active="no"/>
-<layer number="46" name="Milling" color="3" fill="1" visible="yes" active="no"/>
-<layer number="47" name="Measures" color="7" fill="1" visible="yes" active="no"/>
-<layer number="48" name="Document" color="7" fill="1" visible="yes" active="no"/>
-<layer number="49" name="Reference" color="7" fill="1" visible="yes" active="no"/>
-<layer number="50" name="dxf" color="7" fill="1" visible="yes" active="no"/>
-<layer number="51" name="tDocu" color="7" fill="1" visible="yes" active="no"/>
-<layer number="52" name="bDocu" color="7" fill="1" visible="yes" active="no"/>
+<layer number="46" name="Milling" color="3" fill="1" visible="no" active="no"/>
+<layer number="47" name="Measures" color="7" fill="1" visible="no" active="no"/>
+<layer number="48" name="Document" color="7" fill="1" visible="no" active="no"/>
+<layer number="49" name="Reference" color="7" fill="1" visible="no" active="no"/>
+<layer number="50" name="dxf" color="7" fill="1" visible="no" active="no"/>
+<layer number="51" name="tDocu" color="7" fill="1" visible="no" active="no"/>
+<layer number="52" name="bDocu" color="7" fill="1" visible="no" active="no"/>
 <layer number="91" name="Nets" color="2" fill="1" visible="yes" active="yes"/>
 <layer number="92" name="Busses" color="1" fill="1" visible="yes" active="yes"/>
@@
 <instance part="C2" gate="G$1" x="22.86" y="-2.54"/>
 <instance part="C3" gate="G$1" x="30.48" y="-2.54"/>
-<instance part="D1" gate="G$1" x="45.72" y="45.72" rot="R90"/>
+<instance part="D1" gate="G$1" x="43.18" y="45.72" rot="R90"/>
 <instance part="R2" gate="G$1" x="-5.08" y="30.48"/>
 <instance part="R_SENSE" gate="G$1" x="-5.08" y="40.64"/>
@@
 <pinref part="D1" gate="G$1" pin="C"/>
 <wire x1="-10.16" y1="50.8" x2="-10.16" y2="40.64" width="0.1524" layer="91"/>
-<wire x1="45.72" y1="48.26" x2="45.72" y2="50.8" width="0.1524" layer="91"/>
-<wire x1="45.72" y1="50.8" x2="-10.16" y2="50.8" width="0.1524" layer="91"/>
+<wire x1="43.18" y1="48.26" x2="43.18" y2="50.8" width="0.1524" layer="91"/>
+<wire x1="43.18" y1="50.8" x2="-10.16" y2="50.8" width="0.1524" layer="91"/>
 <junction x="-10.16" y="50.8"/>
 <pinref part="IC1" gate="G$1" pin="VCC"/>
@@
 <pinref part="L1" gate="G$1" pin="2"/>
 <pinref part="D1" gate="G$1" pin="A"/>
-<wire x1="35.56" y1="40.64" x2="45.72" y2="40.64" width="0.1524" layer="91"/>
-<wire x1="45.72" y1="40.64" x2="45.72" y2="43.18" width="0.1524" layer="91"/>
+<wire x1="35.56" y1="40.64" x2="43.18" y2="40.64" width="0.1524" layer="91"/>
+<wire x1="43.18" y1="40.64" x2="43.18" y2="43.18" width="0.1524" layer="91"/>
 <pinref part="IC1" gate="G$1" pin="SWC"/>
-<wire x1="35.56" y1="30.48" x2="45.72" y2="30.48" width="0.1524" layer="91"/>
-<wire x1="45.72" y1="30.48" x2="45.72" y2="40.64" width="0.1524" layer="91"/>
-<junction x="45.72" y="40.64"/>
-</segment>
-</net>
+<wire x1="35.56" y1="30.48" x2="43.18" y2="30.48" width="0.1524" layer="91"/>
+<wire x1="43.18" y1="30.48" x2="43.18" y2="40.64" width="0.1524" layer="91"/>
+<junction x="43.18" y="40.64"/>
+</segment>
+</net>

Commit message: Noch ein wenig Layout-Tuning in der LED-Treiberschaltung
Parts:
- removed LED1: 3W, led:LED5MM
- added LED: 3W, pinhead:PINHD-1X2
- C3: device resistor:C-EU025-024X044 -> capacitor-wima:C5/2.5
Connections:
- net N$3: now also LED.1; no longer LED1.A
- net N$4: now also LED.2; no longer LED1.C
Other:
- moved on the sheet: R_SENSE
Changed lines of the file:
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@@
 <part name="GND2" library="supply1" deviceset="GND" device=""/>
 <part name="C2" library="resistor" deviceset="CPOL-EU" device="E2.5-5" value="68µ"/>
-<part name="C3" library="resistor" deviceset="C-EU" device="025-024X044" value="100n"/>
+<part name="C3" library="capacitor-wima" deviceset="C" device="5/2.5" value="100n"/>
 <part name="D1" library="diode" deviceset="SCHOTTKY-DIODE" device="DO35-7" value="MBRS240"/>
 <part name="R2" library="resistor" deviceset="R-EU_" device="0207/10" value="47R"/>
 <part name="R_SENSE" library="resistor" deviceset="R-EU_" device="0207/10" value="0.22R"/>
-<part name="LED1" library="led" deviceset="LED" device="5MM" value="3W"/>
 <part name="L1" library="inductors" deviceset="DR1030" device="" value="220µ"/>
+<part name="LED" library="pinhead" deviceset="PINHD-1X2" device="" value="3W"/>
 </parts>
 <sheets>
@@
 <instance part="D1" gate="G$1" x="43.18" y="45.72" rot="R90"/>
 <instance part="R2" gate="G$1" x="-5.08" y="30.48"/>
-<instance part="R_SENSE" gate="G$1" x="-5.08" y="40.64"/>
-<instance part="LED1" gate="G$1" x="12.7" y="40.64" rot="R90"/>
+<instance part="R_SENSE" gate="G$1" x="-5.08" y="43.18"/>
 <instance part="L1" gate="G$1" x="30.48" y="40.64"/>
+<instance part="LED" gate="G$1" x="17.78" y="40.64"/>
 </instances>
 <busses>
@@
 <pinref part="R_SENSE" gate="G$1" pin="1"/>
 <pinref part="R2" gate="G$1" pin="1"/>
-<wire x1="-10.16" y1="40.64" x2="-10.16" y2="30.48" width="0.1524" layer="91"/>
+<wire x1="-10.16" y1="43.18" x2="-10.16" y2="30.48" width="0.1524" layer="91"/>
 <pinref part="R1" gate="G$1" pin="1"/>
 <wire x1="-10.16" y1="30.48" x2="-10.16" y2="25.4" width="0.1524" layer="91"/>
@@
 <pinref part="SUPPLY1" gate="G$1" pin="VCC"/>
 <wire x1="-10.16" y1="55.88" x2="-10.16" y2="50.8" width="0.1524" layer="91"/>
-<junction x="-10.16" y="40.64"/>
+<junction x="-10.16" y="43.18"/>
 <pinref part="D1" gate="G$1" pin="C"/>
-<wire x1="-10.16" y1="50.8" x2="-10.16" y2="40.64" width="0.1524" layer="91"/>
+<wire x1="-10.16" y1="50.8" x2="-10.16" y2="43.18" width="0.1524" layer="91"/>
 <wire x1="43.18" y1="48.26" x2="43.18" y2="50.8" width="0.1524" layer="91"/>
 <wire x1="43.18" y1="50.8" x2="-10.16" y2="50.8" width="0.1524" layer="91"/>
@@
 <segment>
 <pinref part="R_SENSE" gate="G$1" pin="2"/>
-<pinref part="LED1" gate="G$1" pin="A"/>
-<wire x1="0" y1="40.64" x2="2.54" y2="40.64" width="0.1524" layer="91"/>
+<wire x1="0" y1="43.18" x2="2.54" y2="43.18" width="0.1524" layer="91"/>
 <pinref part="IC1" gate="G$1" pin="IS"/>
-<wire x1="2.54" y1="40.64" x2="10.16" y2="40.64" width="0.1524" layer="91"/>
 <wire x1="5.08" y1="27.94" x2="2.54" y2="27.94" width="0.1524" layer="91"/>
-<wire x1="2.54" y1="27.94" x2="2.54" y2="40.64" width="0.1524" layer="91"/>
-<junction x="2.54" y="40.64"/>
-</segment>
-</net>
-<net name="N$4" class="0">
-<segment>
-<pinref part="LED1" gate="G$1" pin="C"/>
-<pinref part="L1" gate="G$1" pin="1"/>
-<wire x1="17.78" y1="40.64" x2="25.4" y2="40.64" width="0.1524" layer="91"/>
+<wire x1="2.54" y1="27.94" x2="2.54" y2="43.18" width="0.1524" layer="91"/>
+<junction x="2.54" y="43.18"/>
+<pinref part="LED" gate="G$1" pin="1"/>
+<wire x1="2.54" y1="43.18" x2="15.24" y2="43.18" width="0.1524" layer="91"/>
 </segment>
 </net>
@@
 </segment>
 </net>
+<net name="N$4" class="0">
+<segment>
+<pinref part="L1" gate="G$1" pin="1"/>
+<wire x1="15.24" y1="40.64" x2="25.4" y2="40.64" width="0.1524" layer="91"/>
+<pinref part="LED" gate="G$1" pin="2"/>
+</segment>
+</net>

Commit message: R_SENSE angepasst
Parts:
- R_SENSE: value 0.22R -> 0.18R
Other:
- moved on the sheet: C2, C3
Changed lines of the file:
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@@
 <part name="D1" library="diode" deviceset="SCHOTTKY-DIODE" device="DO35-7" value="MBRS240"/>
 <part name="R2" library="resistor" deviceset="R-EU_" device="0207/10" value="47R"/>
-<part name="R_SENSE" library="resistor" deviceset="R-EU_" device="0207/10" value="0.22R"/>
+<part name="R_SENSE" library="resistor" deviceset="R-EU_" device="0207/10" value="0.18R"/>
 <part name="L1" library="inductors" deviceset="DR1030" device="" value="220µ"/>
 <part name="LED" library="pinhead" deviceset="PINHD-1X2" device="" value="3W"/>
@@
 <instance part="C1" gate="G$1" x="43.18" y="22.86"/>
 <instance part="R1" gate="G$1" x="-5.08" y="22.86"/>
-<instance part="SUPPLY2" gate="G$1" x="17.78" y="2.54"/>
-<instance part="GND2" gate="1" x="38.1" y="-10.16"/>
-<instance part="C2" gate="G$1" x="22.86" y="-2.54"/>
-<instance part="C3" gate="G$1" x="30.48" y="-2.54"/>
+<instance part="SUPPLY2" gate="G$1" x="17.78" y="10.16"/>
+<instance part="GND2" gate="1" x="38.1" y="-2.54"/>
+<instance part="C2" gate="G$1" x="22.86" y="5.08"/>
+<instance part="C3" gate="G$1" x="30.48" y="5.08"/>
 <instance part="D1" gate="G$1" x="43.18" y="45.72" rot="R90"/>
 <instance part="R2" gate="G$1" x="-5.08" y="30.48"/>
@@
 <pinref part="SUPPLY2" gate="G$1" pin="VCC"/>
 <pinref part="C2" gate="G$1" pin="+"/>
-<wire x1="17.78" y1="0" x2="22.86" y2="0" width="0.1524" layer="91"/>
+<wire x1="17.78" y1="7.62" x2="22.86" y2="7.62" width="0.1524" layer="91"/>
 <pinref part="C3" gate="G$1" pin="1"/>
-<wire x1="22.86" y1="0" x2="30.48" y2="0" width="0.1524" layer="91"/>
-<junction x="22.86" y="0"/>
+<wire x1="22.86" y1="7.62" x2="30.48" y2="7.62" width="0.1524" layer="91"/>
+<junction x="22.86" y="7.62"/>
 </segment>
 <segment>
@@
 <pinref part="C2" gate="G$1" pin="-"/>
 <pinref part="C3" gate="G$1" pin="2"/>
-<wire x1="22.86" y1="-7.62" x2="30.48" y2="-7.62" width="0.1524" layer="91"/>
+<wire x1="22.86" y1="0" x2="30.48" y2="0" width="0.1524" layer="91"/>
 <pinref part="GND2" gate="1" pin="GND"/>
-<wire x1="30.48" y1="-7.62" x2="38.1" y2="-7.62" width="0.1524" layer="91"/>
-<junction x="30.48" y="-7.62"/>
+<wire x1="30.48" y1="0" x2="38.1" y2="0" width="0.1524" layer="91"/>
+<junction x="30.48" y="0"/>
 </segment>
 </net>

Commit message: Schaltung nochmal angepasst
Parts:
- removed R2: 47R, resistor:R-EU_0207/10
- C1: device resistor:C-EU075-032X103 -> resistor:C-EU050-024X044
- R_SENSE: device resistor:R-EU_0207/10 -> resistor:R-EU_0411/15
Connections:
- removed net N$5: D1.A, IC1.SWC, L1.2
- net N$2: now also D1.A, IC1.SWC, L1.2; no longer R2.2
- net VCC: no longer R2.1
Changed lines of the file:
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@@
 <part name="GND1" library="supply1" deviceset="GND" device=""/>
 <part name="SV1" library="con-lstb" deviceset="MA03-1" device="" value="Control"/>
-<part name="C1" library="resistor" deviceset="C-EU" device="075-032X103" value="330p"/>
+<part name="C1" library="resistor" deviceset="C-EU" device="050-024X044" value="330p"/>
 <part name="R1" library="resistor" deviceset="R-EU_" device="0207/10" value="4.7K"/>
 <part name="SUPPLY2" library="supply2" deviceset="VCC" device=""/>
@@
 <part name="C3" library="capacitor-wima" deviceset="C" device="5/2.5" value="100n"/>
 <part name="D1" library="diode" deviceset="SCHOTTKY-DIODE" device="DO35-7" value="MBRS240"/>
-<part name="R2" library="resistor" deviceset="R-EU_" device="0207/10" value="47R"/>
-<part name="R_SENSE" library="resistor" deviceset="R-EU_" device="0207/10" value="0.18R"/>
+<part name="R_SENSE" library="resistor" deviceset="R-EU_" device="0411/15" value="0.18R"/>
 <part name="L1" library="inductors" deviceset="DR1030" device="" value="220µ"/>
 <part name="LED" library="pinhead" deviceset="PINHD-1X2" device="" value="3W"/>
@@
 <instance part="C3" gate="G$1" x="30.48" y="5.08"/>
 <instance part="D1" gate="G$1" x="43.18" y="45.72" rot="R90"/>
-<instance part="R2" gate="G$1" x="-5.08" y="30.48"/>
 <instance part="R_SENSE" gate="G$1" x="-5.08" y="43.18"/>
 <instance part="L1" gate="G$1" x="30.48" y="40.64"/>
@@
 <segment>
 <pinref part="R_SENSE" gate="G$1" pin="1"/>
-<pinref part="R2" gate="G$1" pin="1"/>
-<wire x1="-10.16" y1="43.18" x2="-10.16" y2="30.48" width="0.1524" layer="91"/>
+<wire x1="-10.16" y1="43.18" x2="-10.16" y2="25.4" width="0.1524" layer="91"/>
 <pinref part="R1" gate="G$1" pin="1"/>
-<wire x1="-10.16" y1="30.48" x2="-10.16" y2="25.4" width="0.1524" layer="91"/>
-<junction x="-10.16" y="30.48"/>
 <wire x1="-10.16" y1="25.4" x2="-10.16" y2="22.86" width="0.1524" layer="91"/>
 <pinref part="SUPPLY1" gate="G$1" pin="VCC"/>
@@
 </segment>
 </net>
-<net name="N$2" class="0">
-<segment>
-<pinref part="IC1" gate="G$1" pin="DC"/>
-<pinref part="R2" gate="G$1" pin="2"/>
-<wire x1="5.08" y1="30.48" x2="0" y2="30.48" width="0.1524" layer="91"/>
-</segment>
-</net>
 <net name="N$3" class="0">
 <segment>
@@
 <pinref part="IC1" gate="G$1" pin="IS"/>
 <wire x1="5.08" y1="27.94" x2="2.54" y2="27.94" width="0.1524" layer="91"/>
-<wire x1="2.54" y1="27.94" x2="2.54" y2="43.18" width="0.1524" layer="91"/>
 <junction x="2.54" y="43.18"/>
 <pinref part="LED" gate="G$1" pin="1"/>
+<wire x1="2.54" y1="27.94" x2="2.54" y2="43.18" width="0.1524" layer="91"/>
 <wire x1="2.54" y1="43.18" x2="15.24" y2="43.18" width="0.1524" layer="91"/>
-</segment>
-</net>
-<net name="N$5" class="0">
-<segment>
-<pinref part="L1" gate="G$1" pin="2"/>
-<pinref part="D1" gate="G$1" pin="A"/>
-<wire x1="35.56" y1="40.64" x2="43.18" y2="40.64" width="0.1524" layer="91"/>
-<wire x1="43.18" y1="40.64" x2="43.18" y2="43.18" width="0.1524" layer="91"/>
-<pinref part="IC1" gate="G$1" pin="SWC"/>
-<wire x1="35.56" y1="30.48" x2="43.18" y2="30.48" width="0.1524" layer="91"/>
-<wire x1="43.18" y1="30.48" x2="43.18" y2="40.64" width="0.1524" layer="91"/>
-<junction x="43.18" y="40.64"/>
 </segment>
 </net>
@@
 </segment>
 </net>
+<net name="N$2" class="0">
+<segment>
+<pinref part="IC1" gate="G$1" pin="DC"/>
+<wire x1="5.08" y1="30.48" x2="5.08" y2="35.56" width="0.1524" layer="91"/>
+<wire x1="5.08" y1="35.56" x2="35.56" y2="35.56" width="0.1524" layer="91"/>
+<pinref part="IC1" gate="G$1" pin="SWC"/>
+<wire x1="35.56" y1="35.56" x2="35.56" y2="30.48" width="0.1524" layer="91"/>
+<pinref part="L1" gate="G$1" pin="2"/>
+<pinref part="D1" gate="G$1" pin="A"/>
+<wire x1="35.56" y1="40.64" x2="43.18" y2="40.64" width="0.1524" layer="91"/>
+<wire x1="43.18" y1="40.64" x2="43.18" y2="43.18" width="0.1524" layer="91"/>
+<wire x1="35.56" y1="35.56" x2="35.56" y2="40.64" width="0.1524" layer="91"/>
+<junction x="35.56" y="35.56"/>
+<junction x="35.56" y="40.64"/>
+</segment>
+</net>
