File: Ampel/controller.sch (EAGLE design)
At the start: 9 parts, among them IC1 ATtiny25, J1 J5MM, X1 22-23-2041

Commit message: spannungsregler
Parts:
- removed J1: J5MM, jumper:J5MM
- added C2: (no value), resistor:C-EU025-024X044
- added C3: (no value), resistor:CPOL-EUE5-4
- added D1, D2: 1N4004, diode:1N4004
- added IC2: 7805L, linear:7805L
- added X2: KUSBVX, con-kycon:KUSBVX
Connections:
- removed net VDD: OUT1.3, OUT2.3, X1-1.S
- new net VEE: C3.+, D1.C, IC2.VI
- net GND: now also C2.2, C3.-, D2.A, IC2.GND, X2.4
- net VCC: now also C2.1, D1.A, D2.C, IC2.VO, OUT1.3, OUT2.3, X2.1; no longer J1.1, J1.2
Changed lines of the file:
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@@
 <part name="GND3" library="supply1" deviceset="GND" device=""/>
 <part name="SUPPLY3" library="supply2" deviceset="VCC" device=""/>
-<part name="SUPPLY4" library="supply2" deviceset="VDD" device=""/>
 <part name="OUT1" library="con-lstb" deviceset="MA03-1" device="" value="RED"/>
 <part name="OUT2" library="con-lstb" deviceset="MA03-1" device="" value="GREEN"/>
 <part name="IN" library="pinhead" deviceset="PINHD-1X3" device="/90"/>
-<part name="SUPPLY5" library="supply2" deviceset="VDD" device=""/>
-<part name="J1" library="jumper" deviceset="J" device="5MM"/>
+<part name="IC2" library="linear" deviceset="78*" device="L" technology="05"/>
+<part name="SUPPLY5" library="supply2" deviceset="VEE" device=""/>
 <part name="SUPPLY6" library="supply2" deviceset="VCC" device=""/>
+<part name="GND4" library="supply1" deviceset="GND" device=""/>
+<part name="C2" library="resistor" deviceset="C-EU" device="025-024X044"/>
+<part name="C3" library="resistor" deviceset="CPOL-EU" device="E5-4"/>
+<part name="D1" library="diode" deviceset="1N4004" device=""/>
+<part name="D2" library="diode" deviceset="1N4004" device=""/>
+<part name="X2" library="con-kycon" deviceset="KUSBVX" device=""/>
+<part name="SUPPLY7" library="supply2" deviceset="VCC" device=""/>
+<part name="GND5" library="supply1" deviceset="GND" device=""/>
 </parts>
 <sheets>
@@
 <instance part="GND3" gate="1" x="81.28" y="15.24"/>
 <instance part="SUPPLY3" gate="G$1" x="88.9" y="12.7" rot="R180"/>
-<instance part="SUPPLY4" gate="G$1" x="88.9" y="33.02"/>
 <instance part="OUT1" gate="G$1" x="33.02" y="-5.08" rot="R90"/>
 <instance part="OUT2" gate="G$1" x="50.8" y="-5.08" rot="R90"/>
 <instance part="IN" gate="A" x="38.1" y="55.88" rot="R90"/>
-<instance part="SUPPLY5" gate="G$1" x="10.16" y="-5.08" rot="R180"/>
-<instance part="J1" gate="1" x="93.98" y="-2.54"/>
-<instance part="SUPPLY6" gate="G$1" x="88.9" y="-10.16" rot="R180"/>
+<instance part="IC2" gate="A1" x="2.54" y="-22.86"/>
+<instance part="SUPPLY5" gate="G$1" x="-20.32" y="-22.86" rot="R90"/>
+<instance part="SUPPLY6" gate="G$1" x="30.48" y="-22.86" rot="R270"/>
+<instance part="GND4" gate="1" x="-22.86" y="-33.02"/>
+<instance part="C2" gate="G$1" x="22.86" y="-25.4"/>
+<instance part="C3" gate="G$1" x="-12.7" y="-25.4"/>
+<instance part="D1" gate="1" x="2.54" y="-15.24" rot="R180"/>
+<instance part="D2" gate="1" x="15.24" y="-25.4" rot="R90"/>
+<instance part="X2" gate="G$1" x="68.58" y="-25.4"/>
+<instance part="SUPPLY7" gate="G$1" x="50.8" y="-20.32" rot="R90"/>
+<instance part="GND5" gate="1" x="50.8" y="-35.56"/>
 </instances>
 <busses>
@@
 <pinref part="C1" gate="G$1" pin="1"/>
 <wire x1="-25.4" y1="30.48" x2="-20.32" y2="30.48" width="0.1524" layer="91"/>
+<pinref part="OUT1" gate="G$1" pin="3"/>
+<wire x1="30.48" y1="7.62" x2="30.48" y2="2.54" width="0.1524" layer="91"/>
+<wire x1="30.48" y1="7.62" x2="48.26" y2="7.62" width="0.1524" layer="91"/>
+<junction x="30.48" y="7.62"/>
+<pinref part="OUT2" gate="G$1" pin="3"/>
+<wire x1="48.26" y1="7.62" x2="48.26" y2="2.54" width="0.1524" layer="91"/>
+<wire x1="30.48" y1="7.62" x2="-30.48" y2="7.62" width="0.1524" layer="91"/>
+<wire x1="-30.48" y1="7.62" x2="-30.48" y2="35.56" width="0.1524" layer="91"/>
+<wire x1="-30.48" y1="35.56" x2="-20.32" y2="35.56" width="0.1524" layer="91"/>
 </segment>
 <segment>
@@
 </segment>
 <segment>
-<pinref part="J1" gate="1" pin="1"/>
-<wire x1="88.9" y1="-7.62" x2="88.9" y2="-2.54" width="0.1524" layer="91"/>
-<wire x1="88.9" y1="-7.62" x2="99.06" y2="-7.62" width="0.1524" layer="91"/>
-<pinref part="J1" gate="1" pin="2"/>
-<wire x1="99.06" y1="-7.62" x2="99.06" y2="-2.54" width="0.1524" layer="91"/>
+<pinref part="IC2" gate="A1" pin="VO"/>
 <pinref part="SUPPLY6" gate="G$1" pin="VCC"/>
-<junction x="88.9" y="-7.62"/>
+<wire x1="12.7" y1="-22.86" x2="15.24" y2="-22.86" width="0.1524" layer="91"/>
+<pinref part="D2" gate="1" pin="C"/>
+<wire x1="15.24" y1="-22.86" x2="22.86" y2="-22.86" width="0.1524" layer="91"/>
+<wire x1="22.86" y1="-22.86" x2="27.94" y2="-22.86" width="0.1524" layer="91"/>
+<junction x="15.24" y="-22.86"/>
+<pinref part="C2" gate="G$1" pin="1"/>
+<junction x="22.86" y="-22.86"/>
+<pinref part="D1" gate="1" pin="A"/>
+<wire x1="5.08" y1="-15.24" x2="15.24" y2="-15.24" width="0.1524" layer="91"/>
+<wire x1="15.24" y1="-15.24" x2="15.24" y2="-22.86" width="0.1524" layer="91"/>
+</segment>
+<segment>
+<pinref part="X2" gate="G$1" pin="1"/>
+<pinref part="SUPPLY7" gate="G$1" pin="VCC"/>
+<wire x1="63.5" y1="-20.32" x2="53.34" y2="-20.32" width="0.1524" layer="91"/>
 </segment>
 </net>
@@
 <wire x1="81.28" y1="22.86" x2="91.44" y2="22.86" width="0.1524" layer="91"/>
 </segment>
+<segment>
+<pinref part="GND4" gate="1" pin="GND"/>
+<wire x1="-22.86" y1="-30.48" x2="-12.7" y2="-30.48" width="0.1524" layer="91"/>
+<pinref part="D2" gate="1" pin="A"/>
+<wire x1="15.24" y1="-27.94" x2="15.24" y2="-30.48" width="0.1524" layer="91"/>
+<pinref part="C3" gate="G$1" pin="-"/>
+<junction x="-12.7" y="-30.48"/>
+<pinref part="IC2" gate="A1" pin="GND"/>
+<wire x1="-12.7" y1="-30.48" x2="2.54" y2="-30.48" width="0.1524" layer="91"/>
+<wire x1="2.54" y1="-30.48" x2="15.24" y2="-30.48" width="0.1524" layer="91"/>
+<junction x="2.54" y="-30.48"/>
+<pinref part="C2" gate="G$1" pin="2"/>
+<wire x1="15.24" y1="-30.48" x2="22.86" y2="-30.48" width="0.1524" layer="91"/>
+<junction x="15.24" y="-30.48"/>
+</segment>
+<segment>
+<pinref part="X2" gate="G$1" pin="4"/>
+<wire x1="63.5" y1="-27.94" x2="50.8" y2="-27.94" width="0.1524" layer="91"/>
+<pinref part="GND5" gate="1" pin="GND"/>
+<wire x1="50.8" y1="-27.94" x2="50.8" y2="-33.02" width="0.1524" layer="91"/>
+</segment>
 </net>
 <net name="RESET" class="0">
@@
 </segment>
 </net>
-<net name="VDD" class="0">
-<segment>
-<pinref part="X1" gate="-1" pin="S"/>
-<wire x1="91.44" y1="25.4" x2="88.9" y2="25.4" width="0.1524" layer="91"/>
-<pinref part="SUPPLY4" gate="G$1" pin="VDD"/>
-<wire x1="88.9" y1="25.4" x2="88.9" y2="30.48" width="0.1524" layer="91"/>
-</segment>
-<segment>
-<pinref part="SUPPLY5" gate="G$1" pin="VDD"/>
-<wire x1="10.16" y1="-2.54" x2="10.16" y2="7.62" width="0.1524" layer="91"/>
-<wire x1="10.16" y1="7.62" x2="30.48" y2="7.62" width="0.1524" layer="91"/>
-<pinref part="OUT1" gate="G$1" pin="3"/>
-<wire x1="30.48" y1="7.62" x2="30.48" y2="2.54" width="0.1524" layer="91"/>
-<wire x1="30.48" y1="7.62" x2="48.26" y2="7.62" width="0.1524" layer="91"/>
-<junction x="30.48" y="7.62"/>
-<pinref part="OUT2" gate="G$1" pin="3"/>
-<wire x1="48.26" y1="7.62" x2="48.26" y2="2.54" width="0.1524" layer="91"/>
-</segment>
-</net>
 <net name="N$1" class="0">
 <segment>
@@
 </segment>
 </net>
+<net name="VEE" class="0">
+<segment>
+<pinref part="SUPPLY5" gate="G$1" pin="VEE"/>
+<pinref part="IC2" gate="A1" pin="VI"/>
+<wire x1="-17.78" y1="-22.86" x2="-12.7" y2="-22.86" width="0.1524" layer="91"/>
+<pinref part="C3" gate="G$1" pin="+"/>
+<wire x1="-12.7" y1="-22.86" x2="-7.62" y2="-22.86" width="0.1524" layer="91"/>
+<junction x="-12.7" y="-22.86"/>
+<pinref part="D1" gate="1" pin="C"/>
+<wire x1="0" y1="-15.24" x2="-12.7" y2="-15.24" width="0.1524" layer="91"/>
+<wire x1="-12.7" y1="-15.24" x2="-12.7" y2="-22.86" width="0.1524" layer="91"/>
+</segment>
+</net>

Commit message: Jumper für Stromversorgung und Spannungsregler angepasst
Parts:
- added JP1: (no value), pinhead:PINHD-1X2
- C2: value (none) -> 0.1µ
- C3: value (none) -> 470µ
- IC2: value 7805L -> 7805TV; device linear:7805L -> linear:7805TV
Connections:
- net GND: now also JP1.1
- net VEE: now also JP1.2
Changed lines of the file:
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@@
 <part name="OUT2" library="con-lstb" deviceset="MA03-1" device="" value="GREEN"/>
 <part name="IN" library="pinhead" deviceset="PINHD-1X3" device="/90"/>
-<part name="IC2" library="linear" deviceset="78*" device="L" technology="05"/>
 <part name="SUPPLY5" library="supply2" deviceset="VEE" device=""/>
 <part name="SUPPLY6" library="supply2" deviceset="VCC" device=""/>
 <part name="GND4" library="supply1" deviceset="GND" device=""/>
-<part name="C2" library="resistor" deviceset="C-EU" device="025-024X044"/>
-<part name="C3" library="resistor" deviceset="CPOL-EU" device="E5-4"/>
+<part name="C2" library="resistor" deviceset="C-EU" device="025-024X044" value="0.1µ"/>
+<part name="C3" library="resistor" deviceset="CPOL-EU" device="E5-4" value="470µ"/>
 <part name="D1" library="diode" deviceset="1N4004" device=""/>
 <part name="D2" library="diode" deviceset="1N4004" device=""/>
@@
 <part name="SUPPLY7" library="supply2" deviceset="VCC" device=""/>
 <part name="GND5" library="supply1" deviceset="GND" device=""/>
+<part name="IC2" library="linear" deviceset="78*" device="TV" technology="05"/>
+<part name="JP1" library="pinhead" deviceset="PINHD-1X2" device=""/>
 </parts>
 <sheets>
@@
 <instance part="OUT2" gate="G$1" x="50.8" y="-5.08" rot="R90"/>
 <instance part="IN" gate="A" x="38.1" y="55.88" rot="R90"/>
-<instance part="IC2" gate="A1" x="2.54" y="-22.86"/>
 <instance part="SUPPLY5" gate="G$1" x="-20.32" y="-22.86" rot="R90"/>
 <instance part="SUPPLY6" gate="G$1" x="30.48" y="-22.86" rot="R270"/>
@@
 <instance part="SUPPLY7" gate="G$1" x="50.8" y="-20.32" rot="R90"/>
 <instance part="GND5" gate="1" x="50.8" y="-35.56"/>
+<instance part="IC2" gate="A1" x="2.54" y="-22.86"/>
+<instance part="JP1" gate="G$1" x="-38.1" y="-27.94" rot="R180"/>
 </instances>
 <busses>
@@
 </segment>
 <segment>
-<pinref part="IC2" gate="A1" pin="VO"/>
 <pinref part="SUPPLY6" gate="G$1" pin="VCC"/>
 <wire x1="12.7" y1="-22.86" x2="15.24" y2="-22.86" width="0.1524" layer="91"/>
@@
 <wire x1="5.08" y1="-15.24" x2="15.24" y2="-15.24" width="0.1524" layer="91"/>
 <wire x1="15.24" y1="-15.24" x2="15.24" y2="-22.86" width="0.1524" layer="91"/>
+<pinref part="IC2" gate="A1" pin="VO"/>
 </segment>
 <segment>
@@
 <pinref part="C3" gate="G$1" pin="-"/>
 <junction x="-12.7" y="-30.48"/>
-<pinref part="IC2" gate="A1" pin="GND"/>
 <wire x1="-12.7" y1="-30.48" x2="2.54" y2="-30.48" width="0.1524" layer="91"/>
+<pinref part="C2" gate="G$1" pin="2"/>
 <wire x1="2.54" y1="-30.48" x2="15.24" y2="-30.48" width="0.1524" layer="91"/>
-<junction x="2.54" y="-30.48"/>
-<pinref part="C2" gate="G$1" pin="2"/>
 <wire x1="15.24" y1="-30.48" x2="22.86" y2="-30.48" width="0.1524" layer="91"/>
 <junction x="15.24" y="-30.48"/>
+<pinref part="IC2" gate="A1" pin="GND"/>
+<junction x="2.54" y="-30.48"/>
+<pinref part="JP1" gate="G$1" pin="1"/>
+<wire x1="-35.56" y1="-30.48" x2="-22.86" y2="-30.48" width="0.1524" layer="91"/>
+<junction x="-22.86" y="-30.48"/>
 </segment>
 <segment>
@@
 <segment>
 <pinref part="SUPPLY5" gate="G$1" pin="VEE"/>
-<pinref part="IC2" gate="A1" pin="VI"/>
 <wire x1="-17.78" y1="-22.86" x2="-12.7" y2="-22.86" width="0.1524" layer="91"/>
 <pinref part="C3" gate="G$1" pin="+"/>
@@
 <wire x1="0" y1="-15.24" x2="-12.7" y2="-15.24" width="0.1524" layer="91"/>
 <wire x1="-12.7" y1="-15.24" x2="-12.7" y2="-22.86" width="0.1524" layer="91"/>
-</segment>
-</net>
+<pinref part="IC2" gate="A1" pin="VI"/>
+<pinref part="JP1" gate="G$1" pin="2"/>
+<wire x1="-35.56" y1="-27.94" x2="-17.78" y2="-27.94" width="0.1524" layer="91"/>
+<wire x1="-17.78" y1="-27.94" x2="-17.78" y2="-22.86" width="0.1524" layer="91"/>
+<junction x="-17.78" y="-22.86"/>
+</segment>
+</net>
