File: power.brd (EAGLE design)
At the start: 14.9 x 34.3 mm, 7 parts, among them IC2 7805TV, X1 22-23-2041

Commit message: Ladekondensatoren angepasst
Parts:
- C3: value 470µ -> 47µ
Changed lines of the file:
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@@
 </element>
 <element name="C2" library="resistor" package="C025-024X044" value="0.1µ" x="11.43" y="16.51" rot="R180"/>
-<element name="C3" library="resistor" package="E5-4" value="470µ" x="8.89" y="25.4"/>
+<element name="C3" library="resistor" package="E5-4" value="47µ" x="8.89" y="25.4"/>
 <element name="D1" library="diode" package="DO41-10" value="1N4004" x="7.62" y="13.97"/>
 <element name="D2" library="diode" package="DO41-10" value="1N4004" x="7.62" y="10.16" rot="R180"/>
@@
 </signal>
 </signals>
-<errors>
-</errors>
 </board>
 </drawing>
