File: power.sch (EAGLE design)
At the start: 7 parts, among them IC2 7805TV, X1 22-23-2041

Commit message: Ladekondensatoren angepasst
Parts:
- C3: value 470µ -> 47µ
Changed lines of the file:
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@@
 <part name="GND4" library="supply1" deviceset="GND" device=""/>
 <part name="C2" library="resistor" deviceset="C-EU" device="025-024X044" value="0.1µ"/>
-<part name="C3" library="resistor" deviceset="CPOL-EU" device="E5-4" value="470µ"/>
+<part name="C3" library="resistor" deviceset="CPOL-EU" device="E5-4" value="47µ"/>
 <part name="D1" library="diode" deviceset="1N4004" device=""/>
 <part name="D2" library="diode" deviceset="1N4004" device=""/>
