File: Schalter/controller.brd (EAGLE design)
At the start: 25.4 x 33.7 mm, 10 parts, among them IC1 ATtiny25

Commit message: Schalter: Ladekondensator eingefügt
Parts:
- added C2: (no value), resistor:E2,5-6
- moved SV1 6.35 mm to (3.81, 12.7)
Connections:
- net GND: now also C2.-
- net VCC: now also C2.+
Routing:
- net VCC: track 21.7 -> 28.9 mm
- net SCK: track 49.2 -> 53.3 mm
- net MOSI: track 33.3 -> 29.5 mm
- net MISO: track 34.9 -> 38.5 mm
- net RESET: track 14.1 -> 11.4 mm
Changed lines of the file:
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@@
 <wire x1="25.39" y1="33.73" x2="0" y2="33.73" width="0" layer="20"/>
 <wire x1="0" y1="33.73" x2="0" y2="0" width="0" layer="20"/>
-<text x="2.54" y="6.35" size="1.016" layer="16" font="vector" rot="MR270" align="bottom-right">CC_BY_SA</text>
+<text x="24.13" y="7.62" size="1.016" layer="16" font="vector" rot="MR270" align="bottom-right">CC_BY_SA</text>
 <hole x="3.81" y="3.81" drill="3.2"/>
 <hole x="3.81" y="29.21" drill="3.2"/>
-<text x="10.16" y="7.62" size="1.016" layer="16" font="vector" rot="MR180" align="bottom-right">Netz39</text>
+<text x="11.43" y="7.62" size="1.016" layer="16" font="vector" rot="MR180" align="bottom-right">Netz39</text>
 </plain>
 <attributes>
@@
 <element name="R1" library="resistor" package="0207/7" value="10K" x="10.16" y="12.7" rot="R270"/>
 <element name="C1" library="resistor" package="C025-024X044" value="10n" x="11.43" y="19.05" rot="R180"/>
-<element name="SV1" library="con-lstb" package="MA03-2" value="ISP" x="3.81" y="19.05" rot="R270">
-<attribute name="OC_NEWARK" value="unknown" x="-13.97" y="0" size="1.778" layer="27" rot="R270" display="off"/>
-<attribute name="MPN" value="" x="-13.97" y="0" size="1.778" layer="27" rot="R270" display="off"/>
-<attribute name="MF" value="" x="-13.97" y="0" size="1.778" layer="27" rot="R270" display="off"/>
-<attribute name="OC_FARNELL" value="unknown" x="-13.97" y="0" size="1.778" layer="27" rot="R270" display="off"/>
+<element name="SV1" library="con-lstb" package="MA03-2" value="ISP" x="3.81" y="12.7" rot="R270">
+<attribute name="OC_NEWARK" value="unknown" x="-13.97" y="-6.35" size="1.778" layer="27" rot="R270" display="off"/>
+<attribute name="MPN" value="" x="-13.97" y="-6.35" size="1.778" layer="27" rot="R270" display="off"/>
+<attribute name="MF" value="" x="-13.97" y="-6.35" size="1.778" layer="27" rot="R270" display="off"/>
+<attribute name="OC_FARNELL" value="unknown" x="-13.97" y="-6.35" size="1.778" layer="27" rot="R270" display="off"/>
 </element>
 <element name="SV2" library="con-lstb" package="MA05-1" value="" x="16.51" y="22.86" rot="R180">
@@
 <attribute name="OC_FARNELL" value="unknown" x="16.51" y="27.94" size="1.778" layer="27" rot="R180" display="off"/>
 </element>
+<element name="C2" library="resistor" package="E2,5-6" value="" x="6.35" y="21.59" rot="R180"/>
 </elements>
 <signals>
@@
 <wire x1="13.97" y1="20.32" x2="12.7" y2="19.05" width="0.8128" layer="16"/>
 <wire x1="12.7" y1="19.05" x2="12.7" y2="16.51" width="0.8128" layer="16"/>
-<wire x1="12.7" y1="16.51" x2="10.16" y2="16.51" width="0.254" layer="16"/>
-<wire x1="10.16" y1="16.51" x2="5.08" y2="21.59" width="0.4064" layer="16"/>
+<wire x1="12.7" y1="16.51" x2="10.16" y2="16.51" width="0.4064" layer="16"/>
 <contactref element="SV3" pad="4"/>
-<wire x1="13.97" y1="22.86" x2="13.97" y2="27.94" width="0.8128" layer="16"/>
+<wire x1="13.97" y1="22.86" x2="13.97" y2="25.4" width="0.8128" layer="16"/>
+<wire x1="13.97" y1="25.4" x2="13.97" y2="27.94" width="0.8128" layer="16"/>
+<wire x1="5.08" y1="15.24" x2="6.35" y2="16.51" width="0.4064" layer="16"/>
+<wire x1="6.35" y1="16.51" x2="10.16" y2="16.51" width="0.4064" layer="16"/>
+<contactref element="C2" pad="+"/>
+<wire x1="9.906" y1="25.4" x2="13.97" y2="25.4" width="0.8128" layer="16"/>
+<wire x1="7.62" y1="21.59" x2="7.62" y2="23.114" width="0.8128" layer="16"/>
+<wire x1="7.62" y1="23.114" x2="9.906" y2="25.4" width="0.8128" layer="16"/>
 </signal>
 <signal name="GND">
@@
 <contactref element="SV2" pad="5"/>
 <contactref element="SV3" pad="5"/>
+<contactref element="C2" pad="-"/>
 </signal>
 <signal name="RESET">
@@
 <contactref element="SV1" pad="5"/>
 <wire x1="12.7" y1="8.89" x2="10.16" y2="8.89" width="0.4064" layer="16"/>
-<wire x1="10.16" y1="8.89" x2="8.89" y2="8.89" width="0.4064" layer="16"/>
-<wire x1="8.89" y1="8.89" x2="2.54" y2="15.24" width="0.4064" layer="16"/>
-<wire x1="2.54" y1="15.24" x2="2.54" y2="16.51" width="0.4064" layer="16"/>
+<wire x1="10.16" y1="8.89" x2="2.54" y2="8.89" width="0.4064" layer="16"/>
+<wire x1="2.54" y1="8.89" x2="2.54" y2="10.16" width="0.4064" layer="16"/>
 </signal>
 <signal name="MISO">
@@
 <contactref element="IC1" pad="6"/>
 <contactref element="SV2" pad="3"/>
-<wire x1="17.78" y1="19.05" x2="17.78" y2="16.51" width="0.4064" layer="16"/>
+<wire x1="17.78" y1="20.32" x2="17.78" y2="16.51" width="0.4064" layer="16"/>
 <wire x1="16.51" y1="22.86" x2="16.51" y2="21.59" width="0.4064" layer="16"/>
-<wire x1="16.51" y1="21.59" x2="17.78" y2="19.05" width="0.4064" layer="16"/>
+<wire x1="16.51" y1="21.59" x2="17.78" y2="20.32" width="0.4064" layer="16"/>
 <contactref element="SV3" pad="3"/>
 <wire x1="16.51" y1="22.86" x2="16.51" y2="27.94" width="0.4064" layer="16"/>
 <wire x1="15.24" y1="30.48" x2="16.51" y2="29.21" width="0.4064" layer="16"/>
 <wire x1="16.51" y1="29.21" x2="16.51" y2="27.94" width="0.4064" layer="16"/>
-<wire x1="2.54" y1="21.59" x2="2.54" y2="22.86" width="0.4064" layer="16"/>
-<wire x1="2.54" y1="22.86" x2="3.81" y2="24.13" width="0.4064" layer="16"/>
-<wire x1="3.81" y1="24.13" x2="8.89" y2="24.13" width="0.4064" layer="16"/>
-<wire x1="8.89" y1="24.13" x2="8.89" y2="29.21" width="0.4064" layer="16"/>
-<wire x1="8.89" y1="29.21" x2="10.16" y2="30.48" width="0.4064" layer="16"/>
+<wire x1="2.54" y1="15.24" x2="2.54" y2="22.86" width="0.4064" layer="16"/>
+<wire x1="2.54" y1="22.86" x2="10.16" y2="30.48" width="0.4064" layer="16"/>
 <wire x1="10.16" y1="30.48" x2="15.24" y2="30.48" width="0.4064" layer="16"/>
 </signal>
@@
 <contactref element="SV2" pad="2"/>
 <wire x1="19.05" y1="22.86" x2="19.05" y2="15.24" width="0.4064" layer="16"/>
-<wire x1="15.24" y1="16.51" x2="15.24" y2="15.24" width="0.254" layer="16"/>
+<wire x1="15.24" y1="16.51" x2="15.24" y2="15.24" width="0.4064" layer="16"/>
 <wire x1="15.24" y1="15.24" x2="16.51" y2="13.97" width="0.4064" layer="16"/>
 <wire x1="16.51" y1="13.97" x2="17.78" y2="13.97" width="0.4064" layer="16"/>
@@
 <contactref element="SV3" pad="2"/>
 <wire x1="19.05" y1="22.86" x2="19.05" y2="27.94" width="0.4064" layer="16"/>
-<wire x1="2.54" y1="19.05" x2="1.27" y2="20.32" width="0.4064" layer="16"/>
-<wire x1="1.27" y1="20.32" x2="1.27" y2="22.86" width="0.4064" layer="16"/>
+<wire x1="2.54" y1="12.7" x2="1.27" y2="13.97" width="0.4064" layer="16"/>
 <wire x1="10.16" y1="31.75" x2="16.51" y2="31.75" width="0.4064" layer="16"/>
 <wire x1="16.51" y1="31.75" x2="19.05" y2="29.21" width="0.4064" layer="16"/>
 <wire x1="19.05" y1="29.21" x2="19.05" y2="27.94" width="0.4064" layer="16"/>
-<wire x1="1.27" y1="22.86" x2="3.81" y2="25.4" width="0.4064" layer="16"/>
-<wire x1="3.81" y1="25.4" x2="7.62" y2="25.4" width="0.4064" layer="16"/>
-<wire x1="7.62" y1="25.4" x2="7.62" y2="29.21" width="0.4064" layer="16"/>
-<wire x1="7.62" y1="29.21" x2="10.16" y2="31.75" width="0.4064" layer="16"/>
+<wire x1="1.27" y1="13.97" x2="1.27" y2="22.86" width="0.4064" layer="16"/>
+<wire x1="1.27" y1="22.86" x2="10.16" y2="31.75" width="0.4064" layer="16"/>
 </signal>
 <signal name="MOSI">
@@
 <wire x1="21.59" y1="22.86" x2="21.59" y2="17.78" width="0.4064" layer="16"/>
 <wire x1="21.59" y1="17.78" x2="20.32" y2="16.51" width="0.4064" layer="16"/>
-<wire x1="20.32" y1="16.51" x2="20.32" y2="13.97" width="0.4064" layer="16"/>
-<wire x1="5.08" y1="19.05" x2="7.62" y2="16.51" width="0.4064" layer="16"/>
-<wire x1="7.62" y1="16.51" x2="7.62" y2="13.97" width="0.4064" layer="16"/>
-<wire x1="7.62" y1="13.97" x2="20.32" y2="13.97" width="0.254" layer="1"/>
 <contactref element="SV3" pad="1"/>
 <wire x1="21.59" y1="22.86" x2="21.59" y2="27.94" width="0.4064" layer="16"/>
-<wire x1="20.32" y1="13.97" x2="20.32" y2="13.97" width="0" layer="19" extent="1-16"/>
-<wire x1="7.62" y1="13.97" x2="7.62" y2="13.97" width="0" layer="19" extent="1-16"/>
+<wire x1="5.08" y1="12.7" x2="17.78" y2="12.7" width="0.4064" layer="16"/>
+<wire x1="17.78" y1="12.7" x2="20.32" y2="15.24" width="0.4064" layer="16"/>
+<wire x1="20.32" y1="15.24" x2="20.32" y2="16.51" width="0.4064" layer="16"/>
 </signal>
 <signal name="N$2">
@@
 <wire x1="15.24" y1="6.35" x2="15.24" y2="8.89" width="0.4064" layer="16"/>
 </signal>
-<signal name="N$3">
-<via x="20.32" y="13.97" extent="1-16" drill="0.8" diameter="1.6764" shape="octagon"/>
-</signal>
-<signal name="N$4">
-<via x="7.62" y="13.97" extent="1-16" drill="0.8" diameter="1.6764" shape="octagon"/>
-</signal>
 <signal name="N$1">
