File: Ampel2/Ampel2.sch (KiCad schematic (older format))
At the start: 20 parts, among them J1 Conn_01x07_Male, J2 Conn_01x07_Male, J3 Conn_01x03_Male, J4 Conn_01x03_Male, J5 AVR-ISP-6, Q1 BC 818-25, Q2 BC 818-25, U1 ATtiny85-20PU

Commit message: Outline and mounting holes
Parts:
- removed C2: 47u, Capacitor_SMD:CP_Elec_4x5.3, symbol Device:CP
- added MK1, MK2, MK3, MK4: 2.0, MountingHole:MountingHole_2.2mm_M2_DIN965, symbol Mechanical:MountingHole
- R2, R4: value 150R -> 100R
- R6, R7, R8: value 33R -> 10R
Changed lines of the file:
@@
 P 4250 6250
 F 0 "R4" H 4320 6296 50  0000 L CNN
-F 1 "150R" H 4320 6205 50  0000 L CNN
+F 1 "100R" H 4320 6205 50  0000 L CNN
 F 2 "Resistor_SMD:R_0603_1608Metric_Pad1.05x0.95mm_HandSolder" V 4180 6250 50  0001 C CNN
 F 3 "~" H 4250 6250 50  0001 C CNN
@@
 P 2250 6200
 F 0 "R2" H 2320 6246 50  0000 L CNN
-F 1 "150R" H 2320 6155 50  0000 L CNN
+F 1 "100R" H 2320 6155 50  0000 L CNN
 F 2 "Resistor_SMD:R_0603_1608Metric_Pad1.05x0.95mm_HandSolder" V 2180 6200 50  0001 C CNN
 F 3 "~" H 2250 6200 50  0001 C CNN
@@
 P 4350 2150
 F 0 "R6" V 4300 1950 50  0000 C CNN
-F 1 "33R" V 4300 2350 50  0000 C CNN
+F 1 "10R" V 4300 2350 50  0000 C CNN
 F 2 "Resistor_SMD:R_0603_1608Metric_Pad1.05x0.95mm_HandSolder" V 4280 2150 50  0001 C CNN
 F 3 "~" H 4350 2150 50  0001 C CNN
@@
 P 4350 2250
 F 0 "R7" V 4300 2050 50  0000 C CNN
-F 1 "33R" V 4300 2450 50  0000 C CNN
+F 1 "10R" V 4300 2450 50  0000 C CNN
 F 2 "Resistor_SMD:R_0603_1608Metric_Pad1.05x0.95mm_HandSolder" V 4280 2250 50  0001 C CNN
 F 3 "~" H 4350 2250 50  0001 C CNN
@@
 P 4350 2350
 F 0 "R8" V 4300 2150 50  0000 C CNN
-F 1 "33R" V 4300 2550 50  0000 C CNN
+F 1 "10R" V 4300 2550 50  0000 C CNN
 F 2 "Resistor_SMD:R_0603_1608Metric_Pad1.05x0.95mm_HandSolder" V 4280 2350 50  0001 C CNN
 F 3 "~" H 4350 2350 50  0001 C CNN
@@
 	1    0    0    -1
 $EndComp
-$Comp
-L Device:CP C2
-U 1 1 5C30264C
-P 6550 5100
-F 0 "C2" H 6668 5146 50  0000 L CNN
-F 1 "47u" H 6668 5055 50  0000 L CNN
-F 2 "Capacitor_SMD:CP_Elec_4x5.3" H 6588 4950 50  0001 C CNN
-F 3 "~" H 6550 5100 50  0001 C CNN
-	1    6550 5100
-	1    0    0    -1
-$EndComp
-$Comp
-L power:+5V #PWR03
-U 1 1 5C302906
-P 6550 4850
-F 0 "#PWR03" H 6550 4700 50  0001 C CNN
-F 1 "+5V" H 6565 5023 50  0000 C CNN
-F 2 "" H 6550 4850 50  0001 C CNN
-F 3 "" H 6550 4850 50  0001 C CNN
-	1    6550 4850
-	1    0    0    -1
-$EndComp
-$Comp
-L power:GND #PWR?
-U 1 1 5C302939
-P 6550 5350
-AR Path="/5C2AB48D/5C302939" Ref="#PWR?"  Part="1"
-AR Path="/5C302939" Ref="#PWR04"  Part="1"
-F 0 "#PWR04" H 6550 5100 50  0001 C CNN
-F 1 "GND" H 6555 5177 50  0000 C CNN
-F 2 "" H 6550 5350 50  0001 C CNN
-F 3 "" H 6550 5350 50  0001 C CNN
-	1    6550 5350
-	1    0    0    -1
-$EndComp
-Wire Wire Line
-	6550 4850 6550 4950
-Wire Wire Line
-	6550 5250 6550 5350
 Text GLabel 10200 3450 2    50   Input ~ 0
 ISP_MISO
+$Comp
+L Mechanical:MountingHole MK1
+U 1 1 5CC1C759
+P 5950 6900
+F 0 "MK1" H 6050 6946 50  0000 L CNN
+F 1 "2.0" H 6050 6855 50  0000 L CNN
+F 2 "MountingHole:MountingHole_2.2mm_M2_DIN965" H 5950 6900 50  0001 C CNN
+F 3 "~" H 5950 6900 50  0001 C CNN
+	1    5950 6900
+	1    0    0    -1
+$EndComp
+$Comp
+L Mechanical:MountingHole MK3
+U 1 1 5CC38696
+P 6400 6900
+F 0 "MK3" H 6500 6946 50  0000 L CNN
+F 1 "2.0" H 6500 6855 50  0000 L CNN
+F 2 "MountingHole:MountingHole_2.2mm_M2_DIN965" H 6400 6900 50  0001 C CNN
+F 3 "~" H 6400 6900 50  0001 C CNN
+	1    6400 6900
+	1    0    0    -1
+$EndComp
+$Comp
+L Mechanical:MountingHole MK2
+U 1 1 5CC3A210
+P 5950 7200
+F 0 "MK2" H 6050 7246 50  0000 L CNN
+F 1 "2.0" H 6050 7155 50  0000 L CNN
+F 2 "MountingHole:MountingHole_2.2mm_M2_DIN965" H 5950 7200 50  0001 C CNN
+F 3 "~" H 5950 7200 50  0001 C CNN
+	1    5950 7200
+	1    0    0    -1
+$EndComp
+$Comp
+L Mechanical:MountingHole MK4
+U 1 1 5CC3A254
+P 6400 7200
+F 0 "MK4" H 6500 7246 50  0000 L CNN
+F 1 "2.0" H 6500 7155 50  0000 L CNN
+F 2 "MountingHole:MountingHole_2.2mm_M2_DIN965" H 6400 7200 50  0001 C CNN
+F 3 "~" H 6400 7200 50  0001 C CNN
+	1    6400 7200
+	1    0    0    -1
+$EndComp
 $EndSCHEMATC

Commit message: Fix Attiny85 footprint
Change to the attiny we actually have (Attiny85V-10 SU)
Parts:
- removed U1: ATtiny85-20PU, Package_SO:SOIC-8_3.9x4.9mm_P1.27mm, symbol MCU_Microchip_ATtiny:ATtiny85-20PU
- added U1: ATtiny85V-10SU, Package_SO:SOIJ-8_5.3x5.3mm_P1.27mm, symbol MCU_Microchip_ATtiny:ATtiny85V-10SU
Connections:
- net +5V: now also U1.8 (VCC)
- net EXT_GN: now also U1.2 (XTAL1/PB3)
- net EXT_RD: now also U1.3 (XTAL2/PB4)
- net GND: now also U1.4 (GND)
- net ISP_MISO: now also U1.6 (PB1)
- net ISP_MOSI: now also U1.5 (AREF/PB0)
- net ISP_RST: now also U1.1 (~RESET~/PB5)
- net ISP_SCK: now also U1.7 (PB2)
Changed lines of the file:
@@
 Wire Wire Line
 	10200 3750 10100 3750
-$Comp
-L MCU_Microchip_ATtiny:ATtiny85-20PU U1
-U 1 1 5C2BE787
-P 2600 2450
-F 0 "U1" H 2070 2496 50  0000 R CNN
-F 1 "ATtiny85-20PU" H 2070 2405 50  0000 R CNN
-F 2 "Package_SO:SOIC-8_3.9x4.9mm_P1.27mm" H 2600 2450 50  0001 C CIN
-F 3 "http://ww1.microchip.com/downloads/en/DeviceDoc/atmel-2586-avr-8-bit-microcontroller-attiny25-attiny45-attiny85_datasheet.pdf" H 2600 2450 50  0001 C CNN
-	1    2600 2450
-	1    0    0    -1
-$EndComp
 Text GLabel 3550 2650 2    50   Input ~ 0
 ISP_RST
@@
 	1    0    0    -1
 $EndComp
+$Comp
+L MCU_Microchip_ATtiny:ATtiny85V-10SU U1
+U 1 1 5C4C79A1
+P 2600 2450
+F 0 "U1" H 2070 2496 50  0000 R CNN
+F 1 "ATtiny85V-10SU" H 2070 2405 50  0000 R CNN
+F 2 "Package_SO:SOIJ-8_5.3x5.3mm_P1.27mm" H 2600 2450 50  0001 C CIN
+F 3 "http://ww1.microchip.com/downloads/en/DeviceDoc/atmel-2586-avr-8-bit-microcontroller-attiny25-attiny45-attiny85_datasheet.pdf" H 2600 2450 50  0001 C CNN
+	1    2600 2450
+	1    0    0    -1
+$EndComp
